File: Coaster_PCB/Team5_Coaster.kicad_pcb (KiCad board)
At the start: 2 copper layers, 54 x 86 mm, 21 parts, among them J1 XT60, J13 3v3, J2 HC-05, J3 10V, J4 Batt, J5 GND, J6 Vin, SW1 SW_SPDT, U1 PicoW

Commit message: Minor PCB change
Routing:
- net Net-(D3-Pad2): track 6.00 -> 6.05 mm, vias 2 -> 0
- net +10V: vias 2 -> 0
Changed lines of the file:
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@@
   (segment (start 103 72.26) (end 105.26 72.26) (width 0.4) (layer "F.Cu") (net 2))
   (segment (start 110 77) (end 110 89) (width 0.4) (layer "F.Cu") (net 2))
-  (via (at 141 127) (size 0.65) (drill 0.3) (layers "F.Cu" "B.Cu") (net 3))
-  (via (at 141 123) (size 0.65) (drill 0.3) (layers "F.Cu" "B.Cu") (net 3))
+  (segment (start 141 123) (end 141 127) (width 0.35) (layer "F.Cu") (net 3))
   (segment (start 142 96) (end 142 72) (width 4) (layer "B.Cu") (net 3))
   (segment (start 107 113) (end 107 94) (width 4) (layer "B.Cu") (net 3))
@@
   (segment (start 107 94) (end 107 70) (width 4) (layer "B.Cu") (net 3))
   (segment (start 106.72 69.72) (end 107 70) (width 2.7) (layer "B.Cu") (net 3))
-  (segment (start 141 123) (end 141 127) (width 1) (layer "B.Cu") (net 3))
   (via (at 149 91) (size 0.65) (drill 0.3) (layers "F.Cu" "B.Cu") (free) (net 4))
   (via (at 101 100) (size 0.65) (drill 0.3) (layers "F.Cu" "B.Cu") (free) (net 4))
@@
   (segment (start 130.841 126.699) (end 131 126.54) (width 6) (layer "B.Cu") (net 11))
   (segment (start 121 126.699) (end 130.841 126.699) (width 6) (layer "B.Cu") (net 11))
-  (via (at 147 130) (size 0.65) (drill 0.3) (layers "F.Cu" "B.Cu") (net 12))
-  (via (at 141 130) (size 0.65) (drill 0.3) (layers "F.Cu" "B.Cu") (net 12))
-  (segment (start 141 130) (end 147 130) (width 1) (layer "B.Cu") (net 12))
+  (segment (start 141 129.925) (end 146.875 129.925) (width 0.35) (layer "F.Cu") (net 12))
+  (segment (start 146.875 129.925) (end 147 129.8) (width 0.35) (layer "F.Cu") (net 12))
   (segment (start 130.985 102.015) (end 130.985 69.015) (width 0.9) (layer "B.Cu") (net 15))
   (segment (start 122 54) (end 115 54) (width 0.8) (layer "B.Cu") (net 15))

Commit message: Post MDR
Python Scripts Debugged. PCB slight changes
Parts:
- added U2: MC79M15_TO220, Package_TO_SOT_THT:TO-220-3_Vertical, F.Cu at (122.0, 86.0)
Routing:
- net +10V: track 106.5 -> 142.9 mm
- net VSYS: track 10.6 -> 42.1 mm
- net GND: vias 186 -> 146
