File: Coaster_PCB/Team5_Coaster.kicad_pcb (KiCad board)
At the start: 2 copper layers, 54 x 86 mm, 22 parts, among them J1 XT60, J13 3v3, J2 HC-05, J3 10V, J4 Batt, J5 GND, J6 Vin, SW1 SW_SPDT, U1 PicoW, U2 MC79M15_TO220

Commit message: Working on CDR Motion PCB
Parts:
- removed D3: LED, LED_SMD:LED_1206_3216Metric
- removed R1: 330, Resistor_SMD:R_1206_3216Metric
- removed Z1: Zener, digikey-footprints:DO-214AC
- moved C1 8.50 mm to (142.0, 121.5), turned to -90 degrees
- moved J6 6.50 mm to (102.2, 127.0), turned to 180 degrees
- moved J1 6.39 mm to (110.2, 130.7), turned to 90 degrees
Routing:
- net +10V: track 142.9 -> 154.1 mm
- net Net-(D3-Pad2): track 6.05 -> 0.00 mm
- net GND: vias 213 -> 205
