File: Coaster_PCB/Team5_Coaster.kicad_sch (KiCad schematic)
At the start: 21 parts, among them J1 XT60, J13 3v3, J2 HC-05, J3 10V, J4 Batt, J5 GND, J6 Vin, SW1 SW_SPDT, U1 PicoW

Commit message: Post MDR
Python Scripts Debugged. PCB slight changes
Parts:
- added U2: MC79M15_TO220, Package_TO_SOT_THT:TO-220-3_Vertical, symbol Regulator_Linear:MC79M15_TO220
Connections:
- net +10V: now also U2.3 (VO)
- net GND: now also U2.1 (GND)
- net VSYS: now also U2.2 (VI)
Changed lines of the file:
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@@
+    (stroke (width 0) (type default) (color 0 0 0 0))
+  )
+  (wire (pts (xy 151.13 115.57) (xy 149.86 115.57))
     (stroke (width 0) (type default) (color 0 0 0 0))
   )
@@
     )
   )
+  (global_label "VSYS" (shape input) (at 134.62 115.57 180) (fields_autoplaced)
+    (effects (font (size 1.27 1.27)) (justify right))
+    (property "Intersheet References" "${INTERSHEET_REFS}" (id 0) (at 127.6107 115.4906 0)
+      (effects (font (size 1.27 1.27)) (justify right) hide)
+    )
+  )
   (global_label "LF2" (shape input) (at 29.21 128.27 180) (fields_autoplaced)
     (effects (font (size 1.27 1.27)) (justify right))
@@
     (pin "1")
   )
+  (symbol (lib_id "power:GND") (at 142.24 107.95 180) (unit 1)
+    (in_bom yes) (on_board yes)
+    (property "Reference" "#PWR0122" (id 0) (at 142.24 101.6 0)
+      (effects (font (size 1.27 1.27)) hide)
+    )
+    (property "Value" "GND" (id 1) (at 142.113 103.5558 0))
+    (property "Footprint" "" (id 2) (at 142.24 107.95 0)
+      (effects (font (size 1.27 1.27)) hide)
+    )
+    (property "Datasheet" "" (id 3) (at 142.24 107.95 0)
+      (effects (font (size 1.27 1.27)) hide)
+    )
+    (pin "1")
+  )
   (symbol (lib_id "Connector_Generic:Conn_01x02") (at 43.18 40.64 180) (unit 1)
     (in_bom yes) (on_board yes)
@@
     (pin "1")
     (pin "2")
+  )
+  (symbol (lib_id "Regulator_Linear:MC79M15_TO220") (at 142.24 115.57 0) (unit 1)
+    (in_bom yes) (on_board yes) (fields_autoplaced)
+    (property "Reference" "U2" (id 0) (at 142.24 120.65 0))
+    (property "Value" "MC79M15_TO220" (id 1) (at 142.24 123.19 0))
+    (property "Footprint" "Package_TO_SOT_THT:TO-220-3_Vertical" (id 2) (at 142.24 120.65 0)
+      (effects (font (size 1.27 1.27) italic) hide)
+    )
+    (property "Datasheet" "http://www.onsemi.com/pub/Collateral/MC79M00-D.PDF" (id 3) (at 142.24 115.57 0)
+      (effects (font (size 1.27 1.27)) hide)
+    )
+    (pin "1")
+    (pin "2")
+    (pin "3")
   )
   (symbol (lib_id "Connector_Generic:Conn_01x02") (at 45.72 53.34 0) (mirror y) (unit 1)
@@
     (pin "9")
   )
+  (symbol (lib_id "power:+10V") (at 151.13 115.57 0) (unit 1)
+    (in_bom yes) (on_board yes)
+    (property "Reference" "#PWR?" (id 0) (at 151.13 119.38 0)
+      (effects (font (size 1.27 1.27)) hide)
+    )
+    (property "Value" "+10V" (id 1) (at 151.511 111.1758 0))
+    (property "Footprint" "" (id 2) (at 151.13 115.57 0)
+      (effects (font (size 1.27 1.27)) hide)
+    )
+    (property "Datasheet" "" (id 3) (at 151.13 115.57 0)
+      (effects (font (size 1.27 1.27)) hide)
+    )
+    (pin "1")
+  )
   (symbol (lib_id "power:GND") (at 34.29 113.03 270) (unit 1)
     (in_bom yes) (on_board yes)
@@
       (reference "#PWR0121") (unit 1) (value "GND") (footprint "")
     )
+    (path "/0ab323da-06dc-4821-92c0-e44483d98e63"
+      (reference "#PWR0122") (unit 1) (value "GND") (footprint "")
+    )
+    (path "/e78f378c-0eb5-422d-a97b-1a258cdab9e2"
+      (reference "#PWR?") (unit 1) (value "+10V") (footprint "")
+    )
     (path "/00000000-0000-0000-0000-000061dd9ea3"
       (reference "C1") (unit 1) (value "2200uF") (footprint "Capacitor_THT:CP_Radial_D10.0mm_P5.00mm")
@@
       (reference "U1") (unit 1) (value "PicoW") (footprint "RPi_Pico:RPi_PicoW_SMD_TH")
     )
+    (path "/252bb8d6-5d41-4d75-bf5f-fe32aebab8f1"
+      (reference "U2") (unit 1) (value "MC79M15_TO220") (footprint "Package_TO_SOT_THT:TO-220-3_Vertical")
+    )
     (path "/00000000-0000-0000-0000-000061df337e"
