File: Team5_Coaster_post_mdr/Team5_Coaster_post_mdr.kicad_pcb (KiCad board)
At the start: 2 copper layers, 21 parts, among them J1 XT60, J13 3v3, J2 HC-05, J3 10V, J5 GND, J6 Vin, SW1 SW_SPDT, U1 PicoW, U2 MC79M15_TO220

Commit message: Working on CDR Motion PCB
Parts:
- added H4: M, MountingHole:MountingHole_4.3mm_M4_Pad_Via, F.Cu at (85.8, 160.5)
- added J10: GND, TestPoint:TestPoint_Plated_Hole_D5.0mm, F.Cu at (148.5, 102.8)
- added J11: GND, TestPoint:TestPoint_Plated_Hole_D5.0mm, F.Cu at (95.5, 131.8)
- added J12: GND, TestPoint:TestPoint_Plated_Hole_D5.0mm, F.Cu at (105.0, 103.0)
- added J14: GND, TestPoint:TestPoint_Plated_Hole_D5.0mm, F.Cu at (158.8, 131.8)
- added J15: GND, TestPoint:TestPoint_Plated_Hole_D5.0mm, F.Cu at (158.2, 67.2)
- added J4: Batt, Connector_PinSocket_2.54mm:PinSocket_1x02_P2.54mm_Vertical, F.Cu at (145.2, 78.3)
- added J7: 10V, TestPoint:TestPoint_Plated_Hole_D5.0mm, F.Cu at (119.2, 134.0)
- added J8: GPIOs, Connector_PinSocket_2.54mm:PinSocket_1x18_P2.54mm_Vertical, F.Cu at (105.2, 66.7)
- added J9: Bluefruit_LE, Connector_PinSocket_2.54mm:PinSocket_1x08_P2.54mm_Vertical, F.Cu at (91.2, 111.5)
- D3: footprint LED_SMD:LED_1206_3216Metric -> LED_THT:LED_D3.0mm
- R1: footprint Resistor_SMD:R_1206_3216Metric -> Resistor_THT:R_Axial_DIN0204_L3.6mm_D1.6mm_P7.62mm_Horizontal
- moved H3 139.5 mm to (168.2, 160.5)
- moved H1 101.3 mm to (85.8, 56.0)
- moved J5 28.3 mm to (96.5, 67.2), turned to 90 degrees
- moved U2 21.4 mm to (124.5, 125.2), turned to 0 degrees
- moved J13 21.2 mm to (155.2, 78.2), turned to 90 degrees
- moved LB1 20.2 mm to (105.7, 118.6)
- moved LF1 20.2 mm to (105.7, 94.8)
- moved U1 19.9 mm to (126.8, 102.8)
- moved RB1 19.8 mm to (147.8, 110.8)
- moved RF1 19.8 mm to (147.8, 87.0)
- moved H2 9.95 mm to (168.2, 56.0)
- moved D3 9.29 mm to (157.8, 151.0), turned to 90 degrees
- moved SW1 6.31 mm to (119.0, 143.1)
- moved D1 6.24 mm to (131.6, 142.7)
- moved J1 6.17 mm to (102.2, 148.8)
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Connections:
- net RX renamed GPIO17
- net TX renamed GPIO16
- U1 pad 1: unconnected-(U1-Pad1) -> DFU
- U1 pad 10: unconnected-(U1-Pad10) -> GPIO7
- U1 pad 11: unconnected-(U1-Pad11) -> GPIO8
- U1 pad 12: unconnected-(U1-Pad12) -> GPIO9
- U1 pad 19: unconnected-(U1-Pad19) -> CTS
- U1 pad 2: unconnected-(U1-Pad2) -> GPIO1
- U1 pad 20: unconnected-(U1-Pad20) -> GPIO15
- U1 pad 29: unconnected-(U1-Pad29) -> GPIO22
- U1 pad 31: unconnected-(U1-Pad31) -> GPIO26
- U1 pad 32: unconnected-(U1-Pad32) -> GPIO27
- U1 pad 34: unconnected-(U1-Pad34) -> GPIO28
- U1 pad 4: unconnected-(U1-Pad4) -> GPIO2
- U1 pad 5: unconnected-(U1-Pad5) -> GPIO3
- U1 pad 6: unconnected-(U1-Pad6) -> GPIO4
- U1 pad 7: unconnected-(U1-Pad7) -> GPIO5
- U1 pad 9: unconnected-(U1-Pad9) -> GPIO6
Routing:
- net +3V3: track 0.00 -> 138.9 mm
- net +10V: track 0.00 -> 128.3 mm
- net GPIO16: track 0.00 -> 117.1 mm
- net GPIO15: track 0.00 -> 106.7 mm
- net GPIO17: track 0.00 -> 105.6 mm
- net CTS: track 0.00 -> 103.8 mm
- net GPIO9: track 0.00 -> 97.4 mm, vias 0 -> 2
- net GPIO8: track 0.00 -> 90.4 mm, vias 0 -> 3
- net GPIO1: track 0.00 -> 67.5 mm, vias 0 -> 1
- net VSYS: track 0.00 -> 59.5 mm
- net GPIO22: track 0.00 -> 51.4 mm
- net DFU: track 0.00 -> 50.6 mm
- net GPIO7: track 0.00 -> 49.8 mm, vias 0 -> 2
- net GPIO26: track 0.00 -> 46.1 mm
- net GPIO6: track 0.00 -> 43.5 mm, vias 0 -> 2
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- added copper zone on F.Cu, net +10V
- added copper zone on B.Cu, net GND
- added copper zone on F.Cu, net GND
- added copper zone on F.Cu, net VCC
Other:
- board outline added: 95 x 117 mm

Commit message: PCB Read for export, DRC passes
Parts:
- J1: value XT60 -> Vin
- SW1: value SW_SPDT -> Vin_Switch
- moved J10 1.75 mm to (150.2, 102.8)
- moved J12 1.75 mm to (103.2, 103.0)
- moved H1 1.60 mm to (84.5, 55.0)
- moved H2 1.46 mm to (169.0, 54.8)
- moved H4 1.46 mm to (84.5, 161.2)
- moved H3 1.06 mm to (169.0, 161.2)
Routing:
- net +3V3: track 138.9 -> 175.4 mm
- net +10V: track 128.3 -> 158.3 mm
- net Net-(D3-Pad2): track 0.00 -> 6.36 mm
- net GPIO9: track 97.4 -> 96.4 mm
- net GPIO8: track 90.4 -> 89.7 mm
- net GND: vias 42 -> 98
Other:
- board size 95 x 117 mm -> 98.1 x 120 mm

Commit message: Updated Pico Symbol, add some silk screen for gpio
Other:
- board text added: "GP0"
- board text added: "GP1"
- board text added: "GP14"
- board text added: "GP15"
- board text added: "GP16"
- board text added: "GP17"
- board text added: "GP2"
- board text added: "GP22"
- board text added: "GP26"
- board text added: "GP27"
- board text added: "GP28"
- board text added: "GP3"
- board text added: "GP4"
- board text added: "GP5"
- board text added: "GP6"
- board text added: "GP7"
- board text added: "GP8"
- board text added: "GP9"
Changed lines of the file:
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@@
     (property "Sheetname" "")
     (attr through_hole)
-    (fp_text reference "U2" (at -3.71 -0.445 90) (layer "F.SilkS")
+    (fp_text reference "U2" (at 2.54 -2.4725 180) (layer "F.SilkS")
       (effects (font (size 1 1) (thickness 0.15)))
     )
@@
       (effects (font (size 0.8 0.8) (thickness 0.15)))
     )
-    (fp_text user "SWDIO" (at 4.5 2.25) (layer "F.SilkS")
-      (effects (font (size 0.8 0.8) (thickness 0.15)))
-    )
     (fp_text user "GP4" (at -12.8 -11.43 45) (layer "F.SilkS")
       (effects (font (size 0.8 0.8) (thickness 0.15)))
@@
     )
     (fp_text user "GP11" (at -13.2 11.7525 45) (layer "F.SilkS")
-      (effects (font (size 0.8 0.8) (thickness 0.15)))
-    )
-    (fp_text user "SWCLK" (at -4 2.25) (layer "F.SilkS")
       (effects (font (size 0.8 0.8) (thickness 0.15)))
     )
@@
     (effects (font (size 1 1) (thickness 0.25)) (justify mirror))
   )
+  (gr_text "GP26" (at 144 64 45) (layer "F.SilkS")
+    (effects (font (size 0.8 0.8) (thickness 0.15)))
+  )
+  (gr_text "GP17" (at 139.25 64 45) (layer "F.SilkS")
+    (effects (font (size 0.8 0.8) (thickness 0.15)))
+  )
+  (gr_text "GP0" (at 105.75 64.25 45) (layer "F.SilkS")
+    (effects (font (size 0.8 0.8) (thickness 0.15)))
+  )
+  (gr_text "GP15" (at 134 64 45) (layer "F.SilkS")
+    (effects (font (size 0.8 0.8) (thickness 0.15)))
+  )
   (gr_text "Omar Areiqat SDP23 Team 5" (at 151.5 154.75) (layer "F.SilkS")
     (effects (font (size 1 1) (thickness 0.25)))
+  )
+  (gr_text "GP14" (at 131.25 64 45) (layer "F.SilkS")
+    (effects (font (size 0.8 0.8) (thickness 0.15)))
+  )
+  (gr_text "GP5" (at 118.25 64.25 45) (layer "F.SilkS")
+    (effects (font (size 0.8 0.8) (thickness 0.15)))
+  )
+  (gr_text "GP1" (at 108.25 64.25 45) (layer "F.SilkS")
+    (effects (font (size 0.8 0.8) (thickness 0.15)))
+  )
+  (gr_text "GP28" (at 149 64 45) (layer "F.SilkS")
+    (effects (font (size 0.8 0.8) (thickness 0.15)))
+  )
+  (gr_text "GP6" (at 121 64.25 45) (layer "F.SilkS")
+    (effects (font (size 0.8 0.8) (thickness 0.15)))
+  )
+  (gr_text "GP8" (at 126 64.25 45) (layer "F.SilkS")
+    (effects (font (size 0.8 0.8) (thickness 0.15)))
+  )
+  (gr_text "GP9" (at 128.5 64.25 45) (layer "F.SilkS")
+    (effects (font (size 0.8 0.8) (thickness 0.15)))
+  )
+  (gr_text "GP2" (at 110.75 64.25 45) (layer "F.SilkS")
+    (effects (font (size 0.8 0.8) (thickness 0.15)))
+  )
+  (gr_text "GP22" (at 141.5 64 45) (layer "F.SilkS")
+    (effects (font (size 0.8 0.8) (thickness 0.15)))
+  )
+  (gr_text "GP4" (at 115.75 64.25 45) (layer "F.SilkS")
+    (effects (font (size 0.8 0.8) (thickness 0.15)))
+  )
+  (gr_text "GP27" (at 146.5 64.25 45) (layer "F.SilkS")
+    (effects (font (size 0.8 0.8) (thickness 0.15)))
+  )
+  (gr_text "GP16" (at 136.5 64 45) (layer "F.SilkS")
+    (effects (font (size 0.8 0.8) (thickness 0.15)))
+  )
+  (gr_text "GP3" (at 113.25 64.25 45) (layer "F.SilkS")
+    (effects (font (size 0.8 0.8) (thickness 0.15)))
+  )
+  (gr_text "GP7" (at 123.25 64.25 45) (layer "F.SilkS")
+    (effects (font (size 0.8 0.8) (thickness 0.15)))
   )
   (segment (start 109.5 96.25) (end 108.05 94.8) (width 0.5) (layer "F.Cu") (net 1))
@@
     (connect_pads (clearance 0.508))
     (min_thickness 0.254) (filled_areas_thickness no)
-    (fill (thermal_gap 0.508) (thermal_bridge_width 0.508))
+    (fill yes (thermal_gap 0.508) (thermal_bridge_width 0.508))
     (polygon
       (pts
@@
     (connect_pads (clearance 0.508))
     (min_thickness 0.254) (filled_areas_thickness no)
-    (fill (thermal_gap 0.508) (thermal_bridge_width 0.508))
+    (fill yes (thermal_gap 0.508) (thermal_bridge_width 0.508))
     (polygon
       (pts
@@
     (connect_pads (clearance 0.508))
     (min_thickness 0.254) (filled_areas_thickness no)
-    (fill (thermal_gap 0.508) (thermal_bridge_width 0.508))
+    (fill yes (thermal_gap 0.508) (thermal_bridge_width 0.508))
     (polygon
       (pts
