File: Coaster_PCB_CDR/Coaster_PCB_CDR.kicad_sch (KiCad schematic)
At the start: 31 parts, among them J1 Vin, J10 Batt, J11 GPIO_14-15, J12 GPIO_27-28, J13 3v3, J18 5v, J19 5v, J2 HC-05, J3 10V, J4 Batt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

Commit message: added jet switches
Parts:
- added SW2, SW?: Vin_Switch, Buggy_Footprints:omar_3pin_switch, symbol Switch:SW_SPDT
- gave numbers to parts that had none: 1
Connections:
- net VCC: now also SW2.1 (A), SW2.2 (B), SW2.3 (C), SW?.1 (A), SW?.2 (B), SW?.3 (C)
Changed lines of the file:
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@@
     (pin "2")
+  )
+  (symbol (lib_id "power:VCC") (at 115.57 69.85 0) (unit 1)
+    (in_bom yes) (on_board yes)
+    (property "Reference" "#PWR?" (id 0) (at 115.57 73.66 0)
+      (effects (font (size 1.27 1.27)) hide)
+    )
+    (property "Value" "VCC" (id 1) (at 115.951 65.4558 0))
+    (property "Footprint" "" (id 2) (at 115.57 69.85 0)
+      (effects (font (size 1.27 1.27)) hide)
+    )
+    (property "Datasheet" "" (id 3) (at 115.57 69.85 0)
+      (effects (font (size 1.27 1.27)) hide)
+    )
+    (pin "1")
   )
   (symbol (lib_id "M5_BuggyProject-rescue:+3.3V-power") (at 116.84 143.51 0) (unit 1)
@@
     (pin "2")
   )
+  (symbol (lib_id "power:VCC") (at 109.22 73.66 0) (unit 1)
+    (in_bom yes) (on_board yes)
+    (property "Reference" "#PWR011" (id 0) (at 109.22 77.47 0)
+      (effects (font (size 1.27 1.27)) hide)
+    )
+    (property "Value" "VCC" (id 1) (at 109.601 69.2658 0))
+    (property "Footprint" "" (id 2) (at 109.22 73.66 0)
+      (effects (font (size 1.27 1.27)) hide)
+    )
+    (property "Datasheet" "" (id 3) (at 109.22 73.66 0)
+      (effects (font (size 1.27 1.27)) hide)
+    )
+    (pin "1")
+  )
   (symbol (lib_id "Connector_Generic:Conn_01x02") (at 127 149.86 270) (unit 1)
     (in_bom yes) (on_board yes)
@@
   (symbol (lib_id "Connector_Generic:Conn_01x01") (at 113.03 127 270) (unit 1)
     (in_bom yes) (on_board yes)
-    (property "Reference" "J?" (id 0) (at 115.062 123.7488 90)
+    (property "Reference" "J7" (id 0) (at 115.062 123.7488 90)
       (effects (font (size 1.27 1.27)) (justify left))
     )
@@
     (pin "1")
     (pin "2")
+  )
+  (symbol (lib_id "power:VCC") (at 125.73 72.39 0) (unit 1)
+    (in_bom yes) (on_board yes)
+    (property "Reference" "#PWR?" (id 0) (at 125.73 76.2 0)
+      (effects (font (size 1.27 1.27)) hide)
+    )
+    (property "Value" "VCC" (id 1) (at 126.111 67.9958 0))
+    (property "Footprint" "" (id 2) (at 125.73 72.39 0)
+      (effects (font (size 1.27 1.27)) hide)
+    )
+    (property "Datasheet" "" (id 3) (at 125.73 72.39 0)
+      (effects (font (size 1.27 1.27)) hide)
+    )
+    (pin "1")
   )
   (symbol (lib_id "power:+5V") (at 102.87 120.65 0) (unit 1)
@@
     (pin "6")
   )
+  (symbol (lib_id "power:VCC") (at 99.06 76.2 0) (unit 1)
+    (in_bom yes) (on_board yes)
+    (property "Reference" "#PWR010" (id 0) (at 99.06 80.01 0)
+      (effects (font (size 1.27 1.27)) hide)
+    )
+    (property "Value" "VCC" (id 1) (at 99.441 71.8058 0))
+    (property "Footprint" "" (id 2) (at 99.06 76.2 0)
+      (effects (font (size 1.27 1.27)) hide)
+    )
+    (property "Datasheet" "" (id 3) (at 99.06 76.2 0)
+      (effects (font (size 1.27 1.27)) hide)
+    )
+    (pin "1")
+  )
   (symbol (lib_id "power:GND") (at 68.58 55.88 0) (unit 1)
     (in_bom yes) (on_board yes)
@@
     )
     (pin "1")
+  )
+  (symbol (lib_id "Switch:SW_SPDT") (at 120.65 72.39 0) (mirror y) (unit 1)
+    (in_bom yes) (on_board yes)
+    (property "Reference" "SW?" (id 0) (at 120.65 68.58 0))
+    (property "Value" "Vin_Switch" (id 1) (at 120.65 77.47 0)
+      (effects (font (size 1.016 1.016)))
+    )
+    (property "Footprint" "Buggy_Footprints:omar_3pin_switch" (id 2) (at 120.65 72.39 0)
+      (effects (font (size 1.27 1.27)) hide)
+    )
+    (property "Datasheet" "~" (id 3) (at 120.65 72.39 0)
+      (effects (font (size 1.27 1.27)) hide)
+    )
+    (pin "1")
+    (pin "2")
+    (pin "3")
   )
   (symbol (lib_id "Regulator_Linear:LM2937xT") (at 123.19 41.91 0) (unit 1)
@@
     (pin "2")
   )
+  (symbol (lib_id "power:VCC") (at 115.57 74.93 0) (unit 1)
+    (in_bom yes) (on_board yes)
+    (property "Reference" "#PWR?" (id 0) (at 115.57 78.74 0)
+      (effects (font (size 1.27 1.27)) hide)
+    )
+    (property "Value" "VCC" (id 1) (at 115.951 70.5358 0))
+    (property "Footprint" "" (id 2) (at 115.57 74.93 0)
+      (effects (font (size 1.27 1.27)) hide)
+    )
+    (property "Datasheet" "" (id 3) (at 115.57 74.93 0)
+      (effects (font (size 1.27 1.27)) hide)
+    )
+    (pin "1")
+  )
   (symbol (lib_id "power:+5V") (at 143.51 143.51 0) (unit 1)
     (in_bom yes) (on_board yes) (fields_autoplaced)
@@
     (pin "1")
   )
+  (symbol (lib_id "Switch:SW_SPDT") (at 104.14 73.66 0) (mirror y) (unit 1)
+    (in_bom yes) (on_board yes)
+    (property "Reference" "SW2" (id 0) (at 104.14 69.85 0))
+    (property "Value" "Vin_Switch" (id 1) (at 104.14 78.74 0)
+      (effects (font (size 1.016 1.016)))
+    )
+    (property "Footprint" "Buggy_Footprints:omar_3pin_switch" (id 2) (at 104.14 73.66 0)
+      (effects (font (size 1.27 1.27)) hide)
+    )
+    (property "Datasheet" "~" (id 3) (at 104.14 73.66 0)
+      (effects (font (size 1.27 1.27)) hide)
+    )
+    (pin "1")
+    (pin "2")
+    (pin "3")
+  )
   (symbol (lib_id "power:GND") (at 69.85 138.43 90) (unit 1)
     (in_bom yes) (on_board yes)
@@
     )
     (property "Datasheet" "" (id 3) (at 69.85 138.43 0)
+      (effects (font (size 1.27 1.27)) hide)
+    )
+    (pin "1")
+  )
+  (symbol (lib_id "power:VCC") (at 99.06 71.12 0) (unit 1)
+    (in_bom yes) (on_board yes)
+    (property "Reference" "#PWR09" (id 0) (at 99.06 74.93 0)
+      (effects (font (size 1.27 1.27)) hide)
+    )
+    (property "Value" "VCC" (id 1) (at 99.441 66.7258 0))
+    (property "Footprint" "" (id 2) (at 99.06 71.12 0)
+      (effects (font (size 1.27 1.27)) hide)
+    )
+    (property "Datasheet" "" (id 3) (at 99.06 71.12 0)
       (effects (font (size 1.27 1.27)) hide)
     )
@@
       (reference "#PWR08") (unit 1) (value "GND") (footprint "")
     )
+    (path "/ce9070c5-1575-4fce-99f1-8526cc6e3001"
+      (reference "#PWR09") (unit 1) (value "VCC") (footprint "")
+    )
+    (path "/81aa9ddc-82de-43a3-8dd2-4c6ecf648a27"
+      (reference "#PWR010") (unit 1) (value "VCC") (footprint "")
+    )
+    (path "/1d8bb3e3-ec85-484f-bb27-ebf6275d494e"
+      (reference "#PWR011") (unit 1) (value "VCC") (footprint "")
+    )
     (path "/abbae294-41f6-434e-be53-e2053185df61"
       (reference "#PWR0101") (unit 1) (value "GND") (footprint "")
@@
       (reference "#PWR0131") (unit 1) (value "+5V") (footprint "")
     )
+    (path "/063f345a-19ea-4ed8-80b8-783a54b6fa7f"
+      (reference "#PWR?") (unit 1) (value "VCC") (footprint "")
+    )
+    (path "/6eb3d3e5-da36-4c31-8065-757a665f317f"
+      (reference "#PWR?") (unit 1) (value "VCC") (footprint "")
+    )
+    (path "/b2ade3fd-2273-46a7-8cfb-1c6f876f500e"
+      (reference "#PWR?") (unit 1) (value "VCC") (footprint "")
+    )
     (path "/00000000-0000-0000-0000-000061dd9ea3"
       (reference "C1") (unit 1) (value "2200uF") (footprint "Capacitor_THT:CP_Radial_D10.0mm_P5.00mm")
@@
       (reference "J6") (unit 1) (value "Vin") (footprint "Connector_PinSocket_2.54mm:PinSocket_1x02_P2.54mm_Vertical")
     )
+    (path "/406bc657-f0d9-4cdc-a558-cd9bffd22dd4"
+      (reference "J7") (unit 1) (value "VCC_Batt") (footprint "TestPoint:TestPoint_Plated_Hole_D5.0mm")
+    )
     (path "/b089b932-0298-427a-aba2-da43d5ed2ba2"
       (reference "J8") (unit 1) (value "GPIO_0-1") (footprint "Connector_PinSocket_2.54mm:PinSocket_1x02_P2.54mm_Vertical")
@@
       (reference "J19") (unit 1) (value "5v") (footprint "Connector_PinSocket_2.54mm:PinSocket_1x02_P2.54mm_Vertical")
     )
-    (path "/406bc657-f0d9-4cdc-a558-cd9bffd22dd4"
-      (reference "J?") (unit 1) (value "VCC_Batt") (footprint "TestPoint:TestPoint_Plated_Hole_D5.0mm")
-    )
     (path "/00000000-0000-0000-0000-000061d32985"
       (reference "LB1") (unit 1) (value "DRV8871") (footprint "Connector_PinSocket_2.54mm:PinSocket_1x04_P2.54mm_Vertical")
@@
       (reference "SW1") (unit 1) (value "Vin_Switch") (footprint "Buggy_Footprints:1101M2S3CQE2")
     )
+    (path "/cae27690-72da-4ed9-b2ec-2fb2cd6d6a73"
+      (reference "SW2") (unit 1) (value "Vin_Switch") (footprint "Buggy_Footprints:omar_3pin_switch")
+    )
+    (path "/99a8fb31-698e-4131-b333-0fa200c7a254"
+      (reference "SW?") (unit 1) (value "Vin_Switch") (footprint "Buggy_Footprints:omar_3pin_switch")
+    )
     (path "/d645b5a5-a402-4a08-b2d8-3b05e5bada03"

Commit message: jet switches
Parts:
- removed H4: M, MountingHole:MountingHole_4.3mm_M4_Pad_Via, symbol Mechanical:MountingHole_Pad
- gave numbers to parts that had none: 1
Connections:
- no-connect marks 14 -> 13
Changed lines of the file:
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@@
   (no_connect (at 92.71 146.05))
   (no_connect (at 69.85 107.95))
-  (no_connect (at 157.48 45.72))
   (no_connect (at 69.85 95.25))
   (no_connect (at 69.85 120.65))
@@
   (symbol (lib_id "power:VCC") (at 115.57 69.85 0) (unit 1)
     (in_bom yes) (on_board yes)
-    (property "Reference" "#PWR?" (id 0) (at 115.57 73.66 0)
+    (property "Reference" "#PWR012" (id 0) (at 115.57 73.66 0)
       (effects (font (size 1.27 1.27)) hide)
     )
@@
   (symbol (lib_id "power:VCC") (at 125.73 72.39 0) (unit 1)
     (in_bom yes) (on_board yes)
-    (property "Reference" "#PWR?" (id 0) (at 125.73 76.2 0)
+    (property "Reference" "#PWR014" (id 0) (at 125.73 76.2 0)
       (effects (font (size 1.27 1.27)) hide)
     )
@@
     (pin "2")
   )
-  (symbol (lib_id "Mechanical:MountingHole_Pad") (at 157.48 43.18 0) (unit 1)
-    (in_bom yes) (on_board yes)
-    (property "Reference" "H4" (id 0) (at 160.02 41.9354 0)
-      (effects (font (size 1.27 1.27)) (justify left))
-    )
-    (property "Value" "M" (id 1) (at 160.02 44.2468 0)
-      (effects (font (size 1.27 1.27)) (justify left))
-    )
-    (property "Footprint" "MountingHole:MountingHole_4.3mm_M4_Pad_Via" (id 2) (at 157.48 43.18 0)
-      (effects (font (size 1.27 1.27)) hide)
-    )
-    (property "Datasheet" "~" (id 3) (at 157.48 43.18 0)
-      (effects (font (size 1.27 1.27)) hide)
-    )
-    (pin "1")
-  )
   (symbol (lib_id "Switch:SW_SPDT") (at 120.65 72.39 0) (mirror y) (unit 1)
     (in_bom yes) (on_board yes)
-    (property "Reference" "SW?" (id 0) (at 120.65 68.58 0))
+    (property "Reference" "SW3" (id 0) (at 120.65 68.58 0))
     (property "Value" "Vin_Switch" (id 1) (at 120.65 77.47 0)
       (effects (font (size 1.016 1.016)))
@@
   (symbol (lib_id "power:VCC") (at 115.57 74.93 0) (unit 1)
     (in_bom yes) (on_board yes)
-    (property "Reference" "#PWR?" (id 0) (at 115.57 78.74 0)
+    (property "Reference" "#PWR013" (id 0) (at 115.57 78.74 0)
       (effects (font (size 1.27 1.27)) hide)
     )
@@
       (reference "#PWR011") (unit 1) (value "VCC") (footprint "")
     )
+    (path "/063f345a-19ea-4ed8-80b8-783a54b6fa7f"
+      (reference "#PWR012") (unit 1) (value "VCC") (footprint "")
+    )
+    (path "/b2ade3fd-2273-46a7-8cfb-1c6f876f500e"
+      (reference "#PWR013") (unit 1) (value "VCC") (footprint "")
+    )
+    (path "/6eb3d3e5-da36-4c31-8065-757a665f317f"
+      (reference "#PWR014") (unit 1) (value "VCC") (footprint "")
+    )
     (path "/abbae294-41f6-434e-be53-e2053185df61"
       (reference "#PWR0101") (unit 1) (value "GND") (footprint "")
@@
       (reference "#PWR0131") (unit 1) (value "+5V") (footprint "")
     )
-    (path "/063f345a-19ea-4ed8-80b8-783a54b6fa7f"
-      (reference "#PWR?") (unit 1) (value "VCC") (footprint "")
-    )
-    (path "/6eb3d3e5-da36-4c31-8065-757a665f317f"
-      (reference "#PWR?") (unit 1) (value "VCC") (footprint "")
-    )
-    (path "/b2ade3fd-2273-46a7-8cfb-1c6f876f500e"
-      (reference "#PWR?") (unit 1) (value "VCC") (footprint "")
-    )
     (path "/00000000-0000-0000-0000-000061dd9ea3"
       (reference "C1") (unit 1) (value "2200uF") (footprint "Capacitor_THT:CP_Radial_D10.0mm_P5.00mm")
@@
       (reference "H3") (unit 1) (value "M") (footprint "MountingHole:MountingHole_4.3mm_M4_Pad_Via")
     )
-    (path "/905ac481-2e05-485f-84fb-07a229113aa2"
-      (reference "H4") (unit 1) (value "M") (footprint "MountingHole:MountingHole_4.3mm_M4_Pad_Via")
-    )
     (path "/00000000-0000-0000-0000-000061de8224"
       (reference "J1") (unit 1) (value "Vin") (footprint "Connector_AMASS:AMASS_XT60-M_1x02_P7.20mm_Vertical")
@@
     )
     (path "/99a8fb31-698e-4131-b333-0fa200c7a254"
-      (reference "SW?") (unit 1) (value "Vin_Switch") (footprint "Buggy_Footprints:omar_3pin_switch")
+      (reference "SW3") (unit 1) (value "Vin_Switch") (footprint "Buggy_Footprints:omar_3pin_switch")
     )
     (path "/d645b5a5-a402-4a08-b2d8-3b05e5bada03"
