File: Coaster_PCB_CDR/_autosave-Coaster_PCB_CDR.kicad_pcb (KiCad board)
At the start: 2 copper layers, 99.5 x 99 mm, 35 parts, among them J1 Vin, J10 GPIO_0-1, J11 5v, J12 5v, J13 GPIO_14-15, J14 5v, J15 GPIO_27-28, J16 5v, J17 5v, J18 5v, J2 Vin, J3 HC-05, J4 HC-05, J5 VCC_Batt, J6 3v3, J7 10V, J8 qwiic, J9 3v3, SW1 Vin_Switch, SW2 Vin_Switch, SW3 Vin_Switch, U1 PicoW, U2 LM2937xT

Commit message: refinements
Parts:
- removed the J18 at (65.0, 120.3)
- added J10: Conn_01x04, Connector_JST:JST_SH_SM04B-SRSS-TB_1x04-1MP_P1.00mm_Horizontal, F.Cu at (137.0, 66.3)
- moved J15 2.63 mm to (84.3, 121.4)
- renumbered J10 to J12, J12 to J13, J13 to J15, J15 to J17, J17 to J18, J5 to J3, J3 to J4, J7 to J5, J4 to J6, J6 to J7, J9 to J8, J8 to J9
Routing:
- net GPIO16: track 101.8 -> 130.4 mm
- net GPIO14: track 28.8 -> 34.7 mm
- net GPIO15: track 29.8 -> 35.1 mm
- net VSYS: track 248.3 -> 249.7 mm
- net GPIO17: track 135.2 -> 134.1 mm
