File: Coaster_PCB_CDR/_autosave-Coaster_PCB_CDR.kicad_sch (KiCad schematic)
At the start: 34 parts, among them J1 Vin, J10 GPIO_0-1, J11 5v, J12 5v, J13 GPIO_14-15, J14 5v, J15 GPIO_27-28, J16 5v, J17 5v, J2 Vin, J3 HC-05, J4 HC-05, J5 VCC_Batt, J6 3v3, J7 10V, J8 qwiic, J9 3v3, SW1 Vin_Switch, SW2 Vin_Switch, SW3 Vin_Switch, U1 PicoW, U2 LM2937xT

Commit message: refinements
Parts:
- added J10: Conn_01x04, Connector_JST:JST_SH_SM04B-SRSS-TB_1x04-1MP_P1.00mm_Horizontal, symbol Connector_Generic:Conn_01x04
- renumbered J10 to J12, J12 to J13, J13 to J15, J15 to J17, J17 to J18, J5 to J3, J3 to J4, J7 to J5, J4 to J6, J6 to J7, J9 to J8, J8 to J9
Connections:
- net +3V3: now also J10.2 (Pin_2)
- net GND: now also J10.1 (Pin_1)
- net GPIO0: now also J10.3 (Pin_3)
- net GPIO1: now also J10.4 (Pin_4)
